File: Pico-CAN-FD-DevBoard/Pico-CAN-FD-DevBoard.kicad_sch (KiCad schematic)
At the start: 55 parts, among them CN1 SM04B-SRSS-TB (LF)(SN), CN2 2601-1102, CN3 2601-1102, CN4 2604-1102, J1 Conn_01x03, J2 Conn_01x08, J3 USB_C_Receptacle_USB2.0_14P, J4 Conn_01x08, SW1 SW_Push, SW2 SW_Push, U1 RP2350B, U2 MCP251863T-H-SS, U3 W25Q128JVS, U4 W25Q128JVS, U5 ESD2CAN24DBZRQ1, U6 TPS51386RJNR, Y1 ABM8-272-T3, Y2 Crystal 40MHz

Commit message: edited things
Connections:
- net ADC0: now also J4.8 (Pin_8)
- net ADC7: now reaches J4.1 (Pin_1)
- net ADC7: now also U1.58 (GPIO47/ADC7)
- net ADC6: now reaches J4.2 (Pin_2)
- net ADC6: now also U1.57 (GPIO46/ADC6)
- net ADC5: now reaches J4.3 (Pin_3)
- net ADC5: now also U1.56 (GPIO45/ADC5)
- net ADC4: now reaches J4.4 (Pin_4)
- net ADC4: now also U1.55 (GPIO44/ADC4)
- net ADC3: now reaches J4.5 (Pin_5)
- net ADC3: now also U1.54 (GPIO43/ADC3)
- net ADC2: now reaches J4.6 (Pin_6)
- net ADC2: now also U1.53 (GPIO42/ADC2)
- net ADC1: now reaches J4.7 (Pin_7)
- net ADC1: now also U1.52 (GPIO41/ADC1)

Commit message: made more changes, enlarged schematic to a2
Parts:
- added J5, J6, J7: Conn_01x03_Socket, Connector_Molex:Molex_SL_171971-0003_1x03_P2.54mm_Vertical, symbol Connector:Conn_01x03_Socket
Connections:
- net GPIO27: now reaches U1.28 (GPIO27)
- net GPIO28: now reaches U1.36 (GPIO28)
- net GPIO29: now reaches U1.37 (GPIO29)
- net GPIO30: now reaches U1.38 (GPIO30)
- net GPIO31: now reaches U1.39 (GPIO31)
- net GPIO32: now reaches U1.40 (GPIO32)
- net GPIO33: now reaches U1.42 (GPIO33)
- net GPIO34: now reaches U1.43 (GPIO34)
- net GPIO35: now reaches U1.44 (GPIO35)
- net GPIO36: now reaches U1.45 (GPIO36)
- net GPIO37: now reaches U1.46 (GPIO37)
- net GPIO38: now reaches U1.47 (GPIO38)
- net GPIO39: now reaches U1.48 (GPIO39)
Other:
- note added: "WAGO"
- moved on the sheet: C10, C14, C15, C16, C17, C18, C19, C20, C21, C22, C23, CN1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

Commit message: added things
Parts:
- removed J4: Conn_01x08, symbol Connector_Generic:Conn_01x08
- removed U6: TPS51386RJNR, TPS51386RJNR:VREG_TPS51386RJNR, symbol TPS51386RJNR:TPS51386RJNR
- added C24, C25: C, symbol Device:C
- added J10, J8: Conn_01x08, symbol Connector_Generic:Conn_01x08
- added J4: Conn_01x10, symbol Connector_Generic:Conn_01x10
- added R14: 110k, symbol Device:R
- added R15: 15k, symbol Device:R
- added U6: TPSM365R6FRDNR, easyeda2kicad:QFN-11_L4.5-W3.5-P0.50-TL_TPSM365R6FRDNR, symbol easyeda2kicad:TPSM365R6FRDNR
Connections:
- net +12V: now also C25.1, U6.2 (EN), U6.3 (VIN)
- net +3V3: now also J5.2 (Pin_2), J6.2 (Pin_2), J7.2 (Pin_2), J10.8 (Pin_8), J4.10 (Pin_10)
- net ADC0: now also J4.9 (Pin_9)
- net ADC1: now also J4.8 (Pin_8)
- net ADC2: now also J4.7 (Pin_7)
- net ADC3: now also J4.6 (Pin_6)
- net ADC4: now also J4.5 (Pin_5)
- net ADC5: now also J4.4 (Pin_4)
- net ADC6: now also J4.3 (Pin_3)
- net ADC7: now also J4.2 (Pin_2)
- net GND: now also J5.3 (Pin_3), J6.3 (Pin_3), J7.3 (Pin_3), C24.2, J4.1 (Pin_1), J8.1 (Pin_1), J8.2 (Pin_2), R15.2, U6.10 (GND), U6.11 (RT/MODE/SYNC)
- net GPIO27: now also J10.7 (Pin_7)
- net GPIO28: now also J10.6 (Pin_6)
- net GPIO29: now also J10.5 (Pin_5)
- net GPIO30: now also J10.4 (Pin_4)
- net GPIO31: now also J10.3 (Pin_3)
- net GPIO32: now also J10.2 (Pin_2)
- net GPIO33: now also J10.1 (Pin_1)
- net GPIO34: now also J8.3 (Pin_3)
- net GPIO35: now also J8.4 (Pin_4)
- net GPIO36: now also J8.5 (Pin_5)
- net GPIO37: now also J8.6 (Pin_6)
- net GPIO38: now also J8.7 (Pin_7)
- net GPIO39: now also J8.8 (Pin_8)
- net GPIO25: now reaches J6.1 (Pin_1)
- net GPIO25: now also U1.26 (GPIO25)
- net GPIO24: now reaches J5.1 (Pin_1)
- net GPIO24: now also U1.25 (GPIO24)
- net GPIO26: now reaches U1.27 (GPIO26)
- net GPIO26: now also J7.1 (Pin_1)
- new net: R14.2, R15.1, U6.9 (FB/BIAS)
- new net: R14.1, U6.4 (VOUT)
- new net: C24.1, U6.8 (VCC)
Other:
- moved on the sheet: CN3

Commit message: added gpio headers, started work on power conversion circuit
Parts:
- added C26: C, symbol Device:C
- added U7: TPSM86638RCGR, SMCJ15A:DIOM7959X262N, symbol easyeda2kicad:TPSM86638RCGR
- C24: value C -> 1u
- C25: value C -> 22u
- R14: value 110k -> 22k
- R15: value 15k -> 10k
Connections:
- net +3V3: now also J10.6 (Pin_6), J10.7 (Pin_7), R14.1, U6.4 (VOUT), C26.1
- net GND: now also C25.2, C26.2
- net 3.3V_PGOOD: now reaches U6.1 (PGOOD)
- net GPIO27: no longer names the net of U1.28 (GPIO27)
- net GPIO27: no longer J10.7 (Pin_7)
- net GPIO28: no longer names the net of U1.36 (GPIO28)
- net GPIO28: no longer J10.6 (Pin_6)
- no-connect marks 1 -> 4
Other:
- note added: "12V to 3.3V buck converter"
- note added: "12V to 5V 6A"
- note added: "ADC Header"
- note added: "Extra GPIO Header"
- note added: "Molex SL GPIO"
- moved on the sheet: C14, C15, C18, C19, C21, C22, C23, C24, C25, CN2, CN3, CN4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

Commit message: more things added
Parts:
- added C27, C28: C, symbol Device:C
- C26: value C -> 22u
Connections:
- net +12V: now also U7.8 (VIN), U7.9 (VIN), C27.1
- net +3V3: now also U7.1 (VOUT), U7.16 (VOUT)
- net GND: now also U7.13 (NC), U7.14 (NC), U7.15 (NC), U7.17 (PGND), U7.18 (PGND), U7.19 (PGND), U7.5 (AGND), C27.2, C28.2
- net 5V_PGOOD: now reaches U7.6 (PG)
- net at U7.7 (SS): now also C28.1
- no-connect marks 4 -> 7
Other:
- note added: "12V to 3.3V 600mA"
- note added: "NC is tied to GND for better thermals"
- note removed: "12V to 3.3V buck converter"
- title: (none) -> Pico-CAN-FD-DevKit

Commit message: changed things
Parts:
- added D1, D2: SMCJ24A_C19077604, easyeda2kicad:SMC_L6.9-W5.9-LS7.9-RD, symbol easyeda2kicad:SMCJ24A_C19077604
- added L2: BLM18PG121SN1D_C14709, easyeda2kicad:L0603, symbol easyeda2kicad:BLM18PG121SN1D_C14709
- added U8: TLV1117-33, Package_TO_SOT_SMD:SOT-223-3_TabPin2, symbol Regulator_Linear:TLV1117-33
Connections:
- net +12V: now also D1.1 (-), D2.1 (-), L2.2; no longer C25.1, U6.2 (EN), U6.3 (VIN)
- net GND: now also D1.2 (+), D2.2 (+)
- new net: C25.1, L2.1, U6.2 (EN), U6.3 (VIN)

Commit message: simplified things
Parts:
- removed C24: 1u, symbol Device:C
- removed C25, C26: 22u, symbol Device:C
- removed J10, J8: Conn_01x08, symbol Connector_Generic:Conn_01x08
- removed J4: Conn_01x10, symbol Connector_Generic:Conn_01x10
- removed L2: BLM18PG121SN1D_C14709, easyeda2kicad:L0603, symbol easyeda2kicad:BLM18PG121SN1D_C14709
- removed R15: 10k, symbol Device:R
- removed U1: RP2350B, Package_DFN_QFN:QFN-80-1EP_10x10mm_P0.4mm_EP3.4x3.4mm, symbol MCU_RaspberryPi:RP2350B
- removed U6: TPSM365R6FRDNR, easyeda2kicad:QFN-11_L4.5-W3.5-P0.50-TL_TPSM365R6FRDNR, symbol easyeda2kicad:TPSM365R6FRDNR
- added D3: LED, LED_SMD:LED_0805_2012Metric, symbol Device:LED
- added D4: WS2812B-2020, LED_SMD:LED_WS2812B-2020_PLCC4_2.0x2.0mm, symbol LED:WS2812B-2020
- added J8: Conn_01x06, symbol Connector_Generic:Conn_01x06
- added R16: 10k, symbol Device:R
- added U9: RP2350A, Package_DFN_QFN:QFN-60-1EP_7x7mm_P0.4mm_EP3.4x3.4mm, symbol MCU_RaspberryPi:RP2350A
- R14: value 22k -> 1k
Connections:
- net GPIO26 is gone; now on net GPIO25: J7.1 (Pin_1)
- net +1V1: now also U9.23 (DVDD), U9.39 (DVDD), U9.50 (VREG_FB), U9.6 (DVDD)
- net +3V3: now also D4.4 (VDD), J8.6 (Pin_6), R16.1, U9.1 (IOVDD), U9.11 (IOVDD), U9.20 (IOVDD), U9.30 (IOVDD), U9.38 (IOVDD), U9.44 (ADC_AVDD), U9.45 (IOVDD), U9.49 (VREG_VIN), U9.53 (USB_OTP_VDD), U9.54 (QSPI_IOVDD); no longer R14.1
- net 5V_PGOOD: now also R16.2
- net ADC0: now also J8.5 (Pin_5)
- net ADC1: now also J8.4 (Pin_4)
- net ADC2: now also J8.3 (Pin_3)
- net ADC3: now also J8.2 (Pin_2)
- net CAN_CS: now also U9.28 (GPIO17)
- net CAN_SCK: now also U9.29 (GPIO18)
- net CAN_SDI: now also U9.27 (GPIO16)
- net CAN_SDO: now also U9.31 (GPIO19)
- net CAN_nINT: now also U9.32 (GPIO20)
- net CAN_nINT0: now also U9.33 (GPIO21)
- net DS1_CLK: now also U9.10 (GPIO7)
- net DS1_DATA: now also U9.9 (GPIO6)
- net GND: now also D3.1 (K), D4.2 (VSS), J8.1 (Pin_1), U9.12 (GPIO8), U9.47 (VREG_PGND), U9.61 (GND)
- net GPIO24: now also J6.1 (Pin_1), U9.36 (GPIO24); no longer J5.1 (Pin_1)
- net GPIO25: now also U9.37 (GPIO25); no longer J6.1 (Pin_1)
- net NPXL_3V3_0: now also U9.4 (GPIO2)
- net NPXL_3V3_1: now also U9.5 (GPIO3)
- net QSPI_CS: now also U9.60 (~{QSPI_SS})
- net QSPI_SCLK: now also U9.56 (QSPI_SCLK)
- net QSPI_SD0: now also U9.57 (QSPI_SD0)
- net QSPI_SD1: now also U9.59 (QSPI_SD1)
- net QSPI_SD2: now also U9.58 (QSPI_SD2)
- net QSPI_SD3: now also U9.55 (QSPI_SD3)
- net RFID_RST: now also U9.18 (GPIO14)
- net SCL: now also U9.3 (GPIO1)
- net SDA: now also U9.2 (GPIO0)
- net SPI_RFID_CS: now also U9.17 (GPIO13)
- net SPI_SCK: now also U9.14 (GPIO10)
- net SPI_SDI: now also U9.16 (GPIO12)
- net SPI_SDO: now also U9.15 (GPIO11)
- net SWCLK: now also U9.24 (SWCLK)
- net SWDIO: now also U9.25 (SWDIO)
- net XIN: now also U9.21 (XIN)
- net XOUT: now also U9.22 (XOUT)
- net at R14.2: now also D3.2 (A)
- net at C14.1, R5.2: now also U9.46 (VREG_AVDD)
- net at R2.2: now also U9.52 (USB_DP)
- net at R10.2, SW2.2: now also U9.26 (RUN)
- net at R1.2: now also U9.51 (USB_DM)
- net at L1.2: now also U9.48 (VREG_LX)
- new net CAN_LED: R14.1, U9.13 (GPIO9)
- new net DS0_CLK: U9.8 (GPIO5)
- new net DS0_DATA: U9.7 (GPIO4)
- new net GPIO22: U9.34 (GPIO22)
- new net GPIO23: J5.1 (Pin_1), U9.35 (GPIO23)
- new net STAT_LED: D4.3 (DIN), U9.19 (GPIO15)
- no-connect marks 7 -> 4
Other:
- note added: "CAN & STAT LED"
- note added: "RP2350A"
- note removed: "12V to 3.3V 600mA"
- note removed: "Extra GPIO Header"
- note removed: "RP2350B"
- moved on the sheet: U8

Commit message: fixed things
Parts:
- added J4: Conn_01x03_Socket, Connector_Molex:Molex_SL_171971-0003_1x03_P2.54mm_Vertical, symbol Connector:Conn_01x03_Socket
Connections:
- net +3V3: now also J4.2 (Pin_2)
- net ADC0: now also U9.40 (GPIO26/ADC0)
- net ADC1: now also U9.41 (GPIO27/ADC1)
- net ADC2: now also U9.42 (GPIO28/ADC2)
- net ADC3: now also U9.43 (GPIO29/ADC3)
- net GND: now also J4.3 (Pin_3)
- net GPIO22: now also J4.1 (Pin_1)
- no-connect marks 4 -> 5
Other:
- moved on the sheet: C10, C14, C15, C16, C17, C18, C19, C20, C21, C22, C23, CN2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
